File: STM32F103_uC_v1/STM32F103_uC_v1.kicad_pcb (KiCad board)
At the start: 4 copper layers, 50.8 x 50.8 mm, 50 parts, among them J1 USB_C_Receptacle, J2 Barrel_Jack, J3 Conn_01x20, J4 Conn_01x20, J5 Screw terminal, J6 Conn_01x04, J7 ST-Link V2, Q1 DMP2120U-7, SW1 SW_Push_Dual, U1 NCP1117LPST33, U2 STM32F103C8Tx, U3 MAX31855, Y1 8MHz, Y2 32.768kHz

Commit message: Finishing touches
Parts:
- moved R14 2.16 mm to (195.1, 80.6)
Connections:
- net /PA11/D- renamed /USB_D-
- net /PA12/D+ renamed /USB_D+
Routing:
- net /USB_D+: track 41.0 -> 61.6 mm
- net VDD: track 65.1 -> 63.3 mm
- net /PB14/MISO2: track 36.0 -> 35.2 mm
- net /PB15/MOSI2: track 38.3 -> 37.6 mm
- net GND: track 130.7 -> 130.6 mm, vias 25 -> 28
- added copper zone on In2.Cu, net /Vin
- added copper zone on In1.Cu, net GND
- added copper zone on In2.Cu, net VDD
- removed copper zone on In1.Cu, net /Vin
- removed copper zone on In2.Cu, net GND
- removed copper zone on In1.Cu, net VDD
